File: fm1608-to-6116.kicad_pcb (KiCad board)
At the start: 2 copper layers, 23.1 x 37.6 mm, 3 parts, among them U1 6116, U2 FM1608

Commit message: Converted to Kicad 8.x
Other:
- net class Default removed
